File: buri-bus-monitor.kicad_pcb (KiCad board)
At the start: 2 copper layers, 99.1 x 158.8 mm, 19 parts, among them P1 Buri-Bus, U1 74HC04, U2 74LS299, U3 74HC00, U4 74HC74, U5 74LS299, U6 74LS299, U7 74LS299, U8 Arduino Nano

Commit message: first pass at layout
Parts:
- added C7: 100n, Capacitors_ThroughHole:C_Disc_D3_P2.5, F.Cu at (63.5, 96.5)
- U2: footprint Housings_DIP:DIP-14_W7.62mm_LongPads -> Housings_DIP:DIP-20_W7.62mm_LongPads
- moved C1 143.2 mm to (48.3, 33.0), turned to 270 degrees
- moved C6 137.6 mm to (61.0, 132.1), turned to 270 degrees
- moved U8 129.3 mm to (85.1, 61.0)
- moved C3 126.8 mm to (73.7, 33.1), turned to 270 degrees
- moved R4 119.8 mm to (59.7, 61.0), turned to 90 degrees
- moved C5 102.9 mm to (96.5, 132.1), turned to 270 degrees
- moved C4 101.8 mm to (99.1, 33.1), turned to 270 degrees
- moved C2 87.8 mm to (96.5, 96.5), turned to 270 degrees
- moved R2 64.3 mm to (52.1, 61.0), turned to 90 degrees
- moved R3 63.3 mm to (55.9, 61.0), turned to 90 degrees
- moved U3 62.7 mm to (78.7, 38.1), turned to 90 degrees
- moved U2 57.3 mm to (101.6, 101.6), turned to 90 degrees
- moved U4 55.9 mm to (104.1, 38.1), turned to 90 degrees
- moved R1 55.2 mm to (48.3, 61.0), turned to 90 degrees
- moved U6 54.6 mm to (66.0, 137.2), turned to 90 degrees
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Routing:
- net +5V: track 0.00 -> 516.7 mm, vias 0 -> 4
- net /~RST: track 0.00 -> 236.8 mm, vias 0 -> 8
- net /RDY: track 0.00 -> 224.0 mm, vias 0 -> 5
- net /R~W: track 0.00 -> 189.0 mm, vias 0 -> 4
- net /~IRQ: track 0.00 -> 185.7 mm, vias 0 -> 4
- net /~AOE: track 0.00 -> 171.5 mm, vias 0 -> 4
- net /SCLK: track 0.00 -> 171.0 mm, vias 0 -> 3
- net /BE: track 0.00 -> 170.2 mm, vias 0 -> 4
- net /PHI2: track 0.00 -> 165.4 mm, vias 0 -> 4
- net /SYNC: track 0.00 -> 158.5 mm, vias 0 -> 4
- net /AS0: track 0.00 -> 145.1 mm, vias 0 -> 4
- net GND: track 0.00 -> 144.9 mm, vias 0 -> 10
- net /D1: track 0.00 -> 138.2 mm, vias 0 -> 4
- net /~NMI: track 0.00 -> 131.3 mm, vias 0 -> 4
- net /AS1: track 0.00 -> 128.6 mm, vias 0 -> 4
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- added copper zone on B.Cu, net GND
